Commit message: Rename robot to husky, and add base_link mesh

File: urdf/husky.gazebo.xacro (robot description, xacro)
@@ -1,4 +1,4 @@
 <?xml version="1.0"?>
-<robot name="mars_explorer" xmlns:xacro="http://ros.org/wiki/xacro">
+<robot name="husky" xmlns:xacro="http://ros.org/wiki/xacro">
   <xacro:arg name="laser_visual"  default="false" />
   <xacro:arg name="camera_visual" default="false"/>
@@ -9,5 +9,5 @@
       <visualize>$(arg imu_visual)</visualize>
       <update_rate>100</update_rate>
-      <topic>model/mars_explorer/imu</topic>
+      <topic>model/husky/imu</topic>
       <gz_frame_id>imu_link</gz_frame_id>
       <imu>
@@ -81,5 +81,5 @@
       <wheel_radius>0.033</wheel_radius>
       <odom_publish_frequency>20</odom_publish_frequency>
-      <topic>model/mars_explorer/cmd_vel</topic>
+      <topic>model/husky/cmd_vel</topic>
       <frame_id>odom</frame_id>
       <child_frame_id>base_link</child_frame_id>
@@ -90,5 +90,5 @@
       filename="ignition-gazebo-joint-state-publisher-system"
       name="ignition::gazebo::systems::JointStatePublisher">
-      <topic>model/mars_explorer/joint_states</topic>
+      <topic>model/husky/joint_states</topic>
     </plugin>
   </gazebo>
@@ -105,5 +105,5 @@
       <pose relative_to='base_scan'>0 0 0 0 0 0</pose>
       <visualize>$(arg laser_visual)</visualize>
-      <topic>model/mars_explorer/scan</topic>
+      <topic>model/husky/scan</topic>
       <update_rate>3</update_rate>
       <gz_frame_id>base_scan</gz_frame_id>
@@ -160,5 +160,5 @@
       <update_rate>10</update_rate>
       <visualize>$(arg camera_visual)</visualize>
-      <topic>/model/mars_explorer/camera</topic>
+      <topic>/model/husky/camera</topic>
       <gz_frame_id>camera_link</gz_frame_id>
     </sensor>

File: urdf/husky.urdf.xacro (robot description, xacro)
@@ -1,6 +1,6 @@
 <?xml version="1.0" ?>
-<robot name="mars_explorer" xmlns:xacro="http://ros.org/wiki/xacro">
+<robot name="husky" xmlns:xacro="http://ros.org/wiki/xacro">
   <xacro:include filename="$(find 41068_ignition_bringup)/urdf/common_properties.urdf.xacro"/>
-  <xacro:include filename="$(find 41068_ignition_bringup)/urdf/mars_explorer.gazebo.xacro"/>
+  <xacro:include filename="$(find 41068_ignition_bringup)/urdf/husky.gazebo.xacro"/>
   <xacro:property name="r200_cam_rgb_px" value="0.005"/>
   <xacro:property name="r200_cam_rgb_py" value="0.018"/>
@@ -17,6 +17,5 @@
       <origin xyz="0 0 0.0" rpy="1.570796 0 1.570796"/>
       <geometry>
-        <!-- <box size="1.0 1.0 0.03"/> -->
-        <mesh filename="file://$(find 41068_ignition_bringup)/urdf/meshes/curiosity_mars_rover.obj" scale="0.37 0.37 0.37"/>
+        <mesh filename="file://$(find 41068_ignition_bringup)/urdf/meshes/base_link.dae"/>
       </geometry>
     </visual>
