Commit message: Begin adding husky model

File: urdf/husky.urdf.xacro (robot description, xacro)
@@ -7,29 +7,82 @@
   <xacro:property name="r200_cam_rgb_pz" value="0.013"/>
   <xacro:property name="r200_cam_depth_offset" value="0.01"/>
-  <link name="base_footprint"/>
-  <joint name="base_joint" type="fixed">
-    <parent link="base_link"/>
-    <child link="base_footprint" />
-    <origin xyz="0 0 -0.010" rpy="0 0 0"/>
-  </joint>
   <link name="base_link">
     <visual>
-      <origin xyz="0 0 0.0" rpy="1.570796 0 1.570796"/>
+      <origin xyz="0 0 0.0" rpy="0 0 0"/>
       <geometry>
         <mesh filename="file://$(find 41068_ignition_bringup)/urdf/meshes/base_link.dae"/>
       </geometry>
-    </visual>
-    <collision>
-      <origin xyz="0 0 0.047" rpy="0 0 0"/>
-      <geometry>
-        <box size="1.0 1.0 0.03"/>
-      </geometry>
-    </collision>
-    <inertial>
-      <origin xyz="0 0 0" rpy="0 0 0"/>
-      <mass value="0"/>
-      <inertia ixx="8.7002718e-03" ixy="-4.7576583e-05" ixz="1.1160499e-04"
-               iyy="8.6195418e-03" iyz="-3.5422299e-06"
-               izz="1.4612727e-02" />
+      <material name="black"/>
+    </visual>
+    <visual name="base_link_fixed_joint_lump__front_bumper_link_visual_3">
+      <origin xyz="0.48 0 0.091" rpy="0 0 0"/>
+      <geometry>
+        <mesh filename="file://$(find 41068_ignition_bringup)/urdf/meshes/bumper.dae"/>
+      </geometry>
+      <material name="black"/>
+    </visual>
+    <visual name="base_link_fixed_joint_lump__rear_bumper_link_visual_4">
+      <origin xyz="-0.48 0 0.091" rpy="0 0 3.14159"/>
+      <geometry>
+        <mesh filename="file://$(find 41068_ignition_bringup)/urdf/meshes/bumper.dae"/>
+      </geometry>
+      <material name="black"/>
+    </visual>
+    <visual name="base_link_fixed_joint_lump__top_chassis_link_visual_5">
+      <origin xyz="0 0 0" rpy="0 0 0"/>
+      <geometry>
+        <mesh filename="file://$(find 41068_ignition_bringup)/urdf/meshes/top_chassis.dae"/>
+      </geometry>
+    </visual>
+    <visual name="base_link_fixed_joint_lump__top_plate_link_visual_6">
+      <origin xyz="0.0812 0 0.245" rpy="0 0 0"/>
+      <geometry>
+        <mesh filename="file://$(find 41068_ignition_bringup)/urdf/meshes/top_plate.dae"/>
+      </geometry>
+      <material name="black"/>
+    </visual>
+    <visual name="base_link_fixed_joint_lump__arch_visual_7">
+      <origin xyz="0.0012 0 0.251" rpy="0 0 0"/>
+      <geometry>
+        <mesh filename="file://$(find 41068_ignition_bringup)/urdf/meshes/jpl04_arch_nosensor.stl"/>
+      </geometry>
+      <material name="black"/>
+    </visual>
+    <collision name="base_link_collision">
+      <origin xyz="0 0 0.12" rpy="0 0 0"/>
+      <geometry>
+        <box size="0.9874 0.5709 0.05"/>
+      </geometry>
+    </collision>
+    <collision name="base_link_collision_bottom">
+      <origin xyz="0 0 0.046" rpy="0 0 0"/>
+      <geometry>
+        <box size="0.80 0.5709 0.095"/>
+      </geometry>
+    </collision>
+    <collision name="base_link_collision_1">
+      <origin xyz="0 0 0.185625" rpy="0 0 0"/>
+      <geometry>
+        <box size="0.78992 0.5709 0.12375"/>
+      </geometry>
+    </collision>
+    <collision name="base_link_fixed_joint_lump__top_plate_link_collision_3">
+      <origin xyz="0.0812 0 0.245" rpy="0 0 0"/>
+      <geometry>
+        <mesh filename="file://$(find 41068_ignition_bringup)/urdf/meshes/top_plate.dae"/>
+      </geometry>
+    </collision>
+    <collision name="base_link_fixed_joint_lump__top_plate_link_collision_4">
+      <origin xyz="0.0812 0 0.245" rpy="0 0 0"/>
+      <geometry>
+        <box size="0.32 0.41 0.09"/>
+      </geometry>
+    </collision>
+    <inertial>
+      <origin xyz="0 0 0.062329" rpy="0 0 0"/>
+      <mass value="46.064"/>
+      <inertia ixx="0.615397" ixy="-0.0240585" ixz="-0.120749"
+               iyy="1.75388" iyz="-0.0028322"
+               izz="2.03641" />
     </inertial>
   </link>

Commit message: Add wheels using xacro macro

File: urdf/husky.urdf.xacro (robot description, xacro)
@@ -3,4 +3,5 @@
   <xacro:include filename="$(find 41068_ignition_bringup)/urdf/common_properties.urdf.xacro"/>
   <xacro:include filename="$(find 41068_ignition_bringup)/urdf/husky.gazebo.xacro"/>
+  <xacro:include filename="$(find 41068_ignition_bringup)/urdf/wheel.urdf.xacro"/>
   <xacro:property name="r200_cam_rgb_px" value="0.005"/>
   <xacro:property name="r200_cam_rgb_py" value="0.018"/>
@@ -87,100 +88,9 @@
     </inertial>
   </link>
-  <joint name="wheel_left_joint" type="continuous">
-    <parent link="base_link"/>
-    <child link="wheel_left_link"/>
-    <origin xyz="0.0 0.144 0.023" rpy="-1.57 0 0"/>
-    <axis xyz="0 0 1"/>
-  </joint>
-  <link name="wheel_left_link">
-    <visual>
-      <origin xyz="0 0 0" rpy="0 0 0"/> <!-- When using tb3 wheel stl, this was rpy="1.57 0 0" -->
-      <geometry>
-        <cylinder length="0.018" radius="0.033"/>
-      </geometry>
-      <material name="dark"/>
-    </visual>
-    <collision>
-      <origin xyz="0 0 0" rpy="0 0 0"/>
-      <geometry>
-        <cylinder length="0.018" radius="0.033"/>
-      </geometry>
-    </collision>
-    <inertial>
-      <origin xyz="0 0 0" />
-      <mass value="2.8498940e-02" />
-      <inertia ixx="1.1175580e-05" ixy="-4.2369783e-11" ixz="-5.9381719e-09"
-               iyy="1.1192413e-05" iyz="-1.4400107e-11"
-               izz="2.0712558e-05" />
-      </inertial>
-  </link>
-  <joint name="wheel_right_joint" type="continuous">
-    <parent link="base_link"/>
-    <child link="wheel_right_link"/>
-    <origin xyz="0.0 -0.144 0.023" rpy="-1.57 0 0"/>
-    <axis xyz="0 0 1"/>
-  </joint>
-  <link name="wheel_right_link">
-    <visual>
-      <origin xyz="0 0 0" rpy="0 0 0"/> <!-- When using tb3 wheel stl, this was rpy="1.57 0 0" -->
-      <geometry>
-        <cylinder length="0.018" radius="0.033"/>
-      </geometry>
-      <material name="dark"/>
-    </visual>
-    <collision>
-      <origin xyz="0 0 0" rpy="0 0 0"/>
-      <geometry>
-        <cylinder length="0.018" radius="0.033"/>
-      </geometry>
-    </collision>
-    <inertial>
-      <origin xyz="0 0 0" />
-      <mass value="2.8498940e-02" />
-      <inertia ixx="1.1175580e-05" ixy="-4.2369783e-11" ixz="-5.9381719e-09"
-               iyy="1.1192413e-05" iyz="-1.4400107e-11"
-               izz="2.0712558e-05" />
-      </inertial>
-  </link>
-  <joint name="caster_back_right_joint" type="fixed">
-    <parent link="base_link"/>
-    <child link="caster_back_right_link"/>
-    <origin xyz="-0.177 -0.064 -0.004" rpy="-1.57 0 0"/>
-  </joint>
-  <link name="caster_back_right_link">
-    <collision>
-      <origin xyz="0 0.001 0" rpy="0 0 0"/>
-      <geometry>
-        <box size="0.030 0.009 0.020"/>
-      </geometry>
-    </collision>
-    <inertial>
-      <origin xyz="0 0 0" />
-      <mass value="0.005" />
-      <inertia ixx="0.001" ixy="0.0" ixz="0.0"
-               iyy="0.001" iyz="0.0"
-               izz="0.001" />
-    </inertial>
-  </link>
-  <joint name="caster_back_left_joint" type="fixed">
-    <parent link="base_link"/>
-    <child link="caster_back_left_link"/>
-    <origin xyz="-0.177 0.064 -0.004" rpy="-1.57 0 0"/>
-  </joint>
-  <link name="caster_back_left_link">
-    <collision>
-      <origin xyz="0 0.001 0" rpy="0 0 0"/>
-      <geometry>
-        <box size="0.030 0.009 0.020"/>
-      </geometry>
-    </collision>
-    <inertial>
-      <origin xyz="0 0 0" />
-      <mass value="0.005" />
-      <inertia ixx="0.001" ixy="0.0" ixz="0.0"
-               iyy="0.001" iyz="0.0"
-               izz="0.001" />
-    </inertial>
-  </link>
+  <!-- Wheels -->
+  <xacro:wheel wheel_id="front_left" x_pos="0.256" y_pos="0.2854"/>
+  <xacro:wheel wheel_id="front_right" x_pos="0.256" y_pos="-0.2854"/>
+  <xacro:wheel wheel_id="rear_left" x_pos="-0.256" y_pos="0.2854"/>
+  <xacro:wheel wheel_id="rear_right" x_pos="-0.256" y_pos="-0.2854"/>
   <joint name="imu_joint" type="fixed">
     <parent link="base_link"/>

Commit message: Paramterise wheels a bit

File: urdf/husky.urdf.xacro (robot description, xacro)
@@ -89,8 +89,8 @@
   </link>
   <!-- Wheels -->
-  <xacro:wheel wheel_id="front_left" x_pos="0.256" y_pos="0.2854"/>
-  <xacro:wheel wheel_id="front_right" x_pos="0.256" y_pos="-0.2854"/>
-  <xacro:wheel wheel_id="rear_left" x_pos="-0.256" y_pos="0.2854"/>
-  <xacro:wheel wheel_id="rear_right" x_pos="-0.256" y_pos="-0.2854"/>
+  <xacro:wheel wheel_id="front_left" x_pos="0.256" y_pos="${wheel_separation/2}"/>
+  <xacro:wheel wheel_id="front_right" x_pos="0.256" y_pos="-${wheel_separation/2}"/>
+  <xacro:wheel wheel_id="rear_left" x_pos="-0.256" y_pos="${wheel_separation/2}"/>
+  <xacro:wheel wheel_id="rear_right" x_pos="-0.256" y_pos="-${wheel_separation/2}"/>
   <joint name="imu_joint" type="fixed">
     <parent link="base_link"/>

File: urdf/wheel.urdf.xacro (robot description, xacro)
@@ -1,4 +1,7 @@
 <?xml version="1.0"?>
 <robot xmlns:xacro="http://www.ros.org/wiki/xacro" name="wheel">
+  <!-- Properties -->
+  <xacro:property name="wheel_separation" value="0.5708"/>
+  <xacro:property name="wheel_radius" value="0.1651"/>
   <xacro:macro name="wheel" params="wheel_id x_pos y_pos">
     <link name="${wheel_id}_wheel_link">
@@ -11,6 +14,7 @@
       <collision>
         <origin xyz="0 0 0" rpy="1.5707963267948966 0 0"/>
+        <contact_coefficients mu="0.5" kp="1+e07" kd="1"/>
         <geometry>
-          <cylinder length="0.1143" radius="0.1651"/>
+          <cylinder length="0.1143" radius="${wheel_radius}"/>
         </geometry>
       </collision>

Commit message: Move lidar, and visualise it in RViz

File: urdf/husky.urdf.xacro (robot description, xacro)
@@ -102,5 +102,5 @@
     <parent link="base_link"/>
     <child link="base_scan"/>
-    <origin xyz="0 0 1.0 " rpy="0 0 0"/>
+    <origin xyz="0 0 0.68" rpy="0 0 0"/>
   </joint>
   <link name="base_scan">
@@ -108,10 +108,10 @@
       <origin xyz="0 0 0" rpy="0 0 0"/>
       <geometry>
-        <cylinder length="0.0315" radius="0.055"/>
+        <cylinder length="0.04" radius="0.09"/>
       </geometry>
       <material name="dark"/>
     </visual>
     <inertial>
-      <mass value="0" /> <!-- 0.114 -->
+      <mass value="0" />
       <origin xyz="0 0 0" />
       <inertia ixx="0.001" ixy="0.0" ixz="0.0"

Commit message: Fix camera

File: urdf/husky.urdf.xacro (robot description, xacro)
@@ -121,5 +121,5 @@
   </link>
   <joint name="camera_joint" type="fixed">
-    <origin xyz="0.5 0.0 0.9" rpy="0 0 0"/> <!-- 0.5 0.0 0.9 -->
+    <origin xyz="0.45 0.0 0.25" rpy="0 0 0"/> <!-- 0.5 0.0 0.9 -->
     <parent link="base_link"/>
     <child link="camera_link"/>
