Commit message: Update parrot.urdf.xacro - merged with parrot thermal

File: urdf_drone/parrot.urdf.xacro (robot description, xacro)
@@ -1,107 +1,101 @@
 <?xml version="1.0" ?>
-<robot name="parrot" xmlns:xacro="http://ros.org/wiki/xacro">
-  <xacro:include filename="$(find 41068_ignition_bringup)/urdf_drone/common_properties.urdf.xacro"/>
-  <xacro:include filename="$(find 41068_ignition_bringup)/urdf_drone/parrot.gazebo.xacro"/>
+<robot name="parrot" xmlns:xacro="http://www.ros.org/wiki/xacro">
+  <!-- === Includes: use your package (change if merging elsewhere) === -->
+  <xacro:include filename="$(find thermal_detection)/urdf_drone/common_properties.urdf.xacro"/>
+  <xacro:include filename="$(find thermal_detection)/urdf_drone/parrot.gazebo.xacro"/>
+  <!-- === Asset root so mesh paths are easy to switch ===
+       If you want to keep meshes in 41068_ignition_bringup, set:
+       asset_root = '$(find 41068_ignition_bringup)/urdf_drone'
+  -->
+  <xacro:property name="asset_root" value="$(find thermal_detection)/urdf_drone"/>
+  <!-- Camera placement helpers (same as both versions) -->
   <xacro:property name="r200_cam_rgb_px" value="0.005"/>
   <xacro:property name="r200_cam_rgb_py" value="0.018"/>
   <xacro:property name="r200_cam_rgb_pz" value="0.013"/>
   <xacro:property name="r200_cam_depth_offset" value="0.01"/>
-  <!-- Main link -->
+  <!-- =============== Base hull =============== -->
   <link name="base_link">
     <inertial>
       <origin xyz="0 0 0" rpy="0 0 0"/>
-      <mass value="0.503"/> <!-- kg -->
-      <inertia ixx="1.805e-3" ixy="-8.619e-7" ixz="1.555e-5"
-               iyy="1.764e-3" iyz="3.595e-7"
-               izz="3.328e-3" />
+      <mass value="0.503"/>
+      <inertia
+        ixx="1.805e-3" ixy="-8.619e-7" ixz="1.555e-5"
+        iyy="1.764e-3" iyz="3.595e-7"
+        izz="3.328e-3"/>
     </inertial>
-<!--     <collision name="collision">
+    <!-- (Optional) simple collision box, keep commented unless you need it
+    <collision name="collision">
       <origin xyz="-0.00424 0.00014 -0.00595" rpy="0 0 0"/>
-      <geometry>
-        <box size="0.5 0.5 0.2"/>
-      </geometry>
-    </collision> -->
+      <geometry><box size="0.5 0.5 0.2"/></geometry>
+    </collision>
+    -->
     <visual name="hull">
-      <geometry>
-        <mesh filename="file://$(find 41068_ignition_bringup)/urdf_drone/meshes/hull.dae"/>
-      </geometry>
+      <geometry><mesh filename="file://${asset_root}/meshes/hull.dae"/></geometry>
     </visual>
     <visual name="propeller_rr">
-      <origin xyz="-0.09035 -0.11423 -0.00501" rpy="0 0 0"/>
-      <geometry>
-        <mesh filename="file://$(find 41068_ignition_bringup)/urdf_drone/meshes/propeller_rr.dae"/>
-      </geometry>
+      <origin xyz="-0.09035 -0.11423 -0.00501"/>
+      <geometry><mesh filename="file://${asset_root}/meshes/propeller_rr.dae"/></geometry>
     </visual>
     <visual name="propeller_rl">
-      <origin xyz="0.09035 0.11452 -0.00501" rpy="0 0 0"/>
-      <geometry>
-        <mesh filename="file://$(find 41068_ignition_bringup)/urdf_drone/meshes/propeller_rl.dae"/>
-      </geometry>
+      <origin xyz="0.09035 0.11452 -0.00501"/>
+      <geometry><mesh filename="file://${asset_root}/meshes/propeller_rl.dae"/></geometry>
     </visual>
     <visual name="propeller_fr">
-      <origin xyz="0.08456 -0.11435 -0.00501" rpy="0 0 0"/>
-      <geometry>
-        <mesh filename="file://$(find 41068_ignition_bringup)/urdf_drone/meshes/propeller_fr.dae"/>
-      </geometry>
+      <origin xyz="0.08456 -0.11435 -0.00501"/>
+      <geometry><mesh filename="file://${asset_root}/meshes/propeller_fr.dae"/></geometry>
     </visual>
     <visual name="propeller_fl">
-      <origin xyz="0.08456 0.11463 -0.00501" rpy="0 0 0"/>
-      <geometry>
-        <mesh filename="file://$(find 41068_ignition_bringup)/urdf_drone/meshes/propeller_fl.dae"/>
-      </geometry>
+      <origin xyz="0.08456 0.11463 -0.00501"/>
+      <geometry><mesh filename="file://${asset_root}/meshes/propeller_fl.dae"/></geometry>
     </visual>
   </link>
+  <!-- =============== IMU =============== -->
   <joint name="imu_joint" type="fixed">
     <parent link="base_link"/>
-    <child link="imu_link"/>
-    <origin xyz="0.0 0 0.068" rpy="0 0 0"/>
+    <child  link="imu_link"/>
+    <origin xyz="0.0 0 0.068"/>
   </joint>
   <link name="imu_link"/>
+  <!-- =============== Lidar puck (viz) =============== -->
   <joint name="scan_joint" type="fixed">
     <parent link="base_link"/>
-    <child link="base_scan"/>
-    <origin xyz="0 0 0.2" rpy="0 0 0"/>
+    <child  link="base_scan"/>
+    <origin xyz="0 0 0.2"/>
   </joint>
   <link name="base_scan">
     <visual>
-      <origin xyz="0 0 0" rpy="0 0 0"/>
-      <geometry>
-        <cylinder length="0.04" radius="0.09"/>
-      </geometry>
+      <origin xyz="0 0 0"/>
+      <geometry><cylinder length="0.04" radius="0.09"/></geometry>
       <material name="dark"/>
     </visual>
     <inertial>
-      <mass value="0" />
-      <origin xyz="0 0 0" />
-      <inertia ixx="0.001" ixy="0.0" ixz="0.0"
-               iyy="0.001" iyz="0.0"
-               izz="0.001" />
+      <mass value="0"/>
+      <origin xyz="0 0 0"/>
+      <inertia ixx="0.001" ixy="0.0" ixz="0.0" iyy="0.001" iyz="0.0" izz="0.001"/>
     </inertial>
   </link>
+  <!-- =============== Camera mast =============== -->
   <joint name="camera_joint" type="fixed">
-    <origin xyz="0.25 0.0 0.25" rpy="0 0.785398 0"/> <!-- 0.5 0.0 0.9 -->
+    <origin xyz="0.25 0.0 0.25" rpy="0 0.785398 0"/>
     <parent link="base_link"/>
-    <child link="camera_link"/>
+    <child  link="camera_link"/>
   </joint>
   <link name="camera_link">
     <visual>
-     <origin xyz="0 0 0" rpy="0 0 0"/>
-      <geometry>
-        <box size="0.02 0.08 0.05"/>
-      </geometry>
+      <origin xyz="0 0 0"/>
+      <geometry><box size="0.02 0.08 0.05"/></geometry>
       <material name="dark"/>
     </visual>
     <visual>
-     <origin xyz="0.015 0 0" rpy="0 1.57 0"/>
-      <geometry>
-        <cylinder length="0.03" radius="0.02"/>
-      </geometry>
+      <origin xyz="0.015 0 0" rpy="0 1.57 0"/>
+      <geometry><cylinder length="0.03" radius="0.02"/></geometry>
       <material name="dark"/>
     </visual>
   </link>
+  <!-- =============== RGB frames =============== -->
   <joint name="camera_rgb_joint" type="fixed">
-    <origin xyz="${r200_cam_rgb_px} ${r200_cam_rgb_py} ${r200_cam_rgb_pz}" rpy="0 0 0"/>
+    <origin xyz="${r200_cam_rgb_px} ${r200_cam_rgb_py} ${r200_cam_rgb_pz}"/>
     <parent link="camera_link"/>
-    <child link="camera_rgb_frame"/>
+    <child  link="camera_rgb_frame"/>
   </joint>
   <link name="camera_rgb_frame"/>
@@ -109,11 +103,12 @@
     <origin xyz="0 0 0" rpy="-1.57 0 -1.57"/>
     <parent link="camera_rgb_frame"/>
-    <child link="camera_rgb_optical_frame"/>
+    <child  link="camera_rgb_optical_frame"/>
   </joint>
   <link name="camera_rgb_optical_frame"/>
+  <!-- =============== Depth frames =============== -->
   <joint name="camera_depth_joint" type="fixed">
-    <origin xyz="${r200_cam_rgb_px} ${r200_cam_rgb_py + r200_cam_depth_offset} ${r200_cam_rgb_pz}" rpy="0 0 0"/>
+    <origin xyz="${r200_cam_rgb_px} ${r200_cam_rgb_py + r200_cam_depth_offset} ${r200_cam_rgb_pz}"/>
     <parent link="camera_link"/>
-    <child link="camera_depth_frame"/>
+    <child  link="camera_depth_frame"/>
   </joint>
   <link name="camera_depth_frame"/>
@@ -121,6 +116,8 @@
     <origin xyz="0 0 0" rpy="-1.57 0 -1.57"/>
     <parent link="camera_depth_frame"/>
-    <child link="camera_depth_optical_frame"/>
+    <child  link="camera_depth_optical_frame"/>
   </joint>
   <link name="camera_depth_optical_frame"/>
+  <!-- =============== Add Gazebo sensors + thermal cam =============== -->
+  <xacro:parrot_gz_extensions/>
 </robot>

Commit message: Update parrot.urdf.xacro - better implementation

File: urdf_drone/parrot.urdf.xacro (robot description, xacro)
@@ -1,13 +1,10 @@
 <?xml version="1.0" ?>
 <robot name="parrot" xmlns:xacro="http://www.ros.org/wiki/xacro">
-  <!-- === Includes: use your package (change if merging elsewhere) === -->
-  <xacro:include filename="$(find thermal_detection)/urdf_drone/common_properties.urdf.xacro"/>
-  <xacro:include filename="$(find thermal_detection)/urdf_drone/parrot.gazebo.xacro"/>
-  <!-- === Asset root so mesh paths are easy to switch ===
-       If you want to keep meshes in 41068_ignition_bringup, set:
-       asset_root = '$(find 41068_ignition_bringup)/urdf_drone'
-  -->
-  <xacro:property name="asset_root" value="$(find thermal_detection)/urdf_drone"/>
-  <!-- Camera placement helpers (same as both versions) -->
+  <!-- Use your ignition package for includes -->
+  <xacro:include filename="$(find 41068_ignition_bringup)/urdf_drone/common_properties.urdf.xacro"/>
+  <xacro:include filename="$(find 41068_ignition_bringup)/urdf_drone/parrot.gazebo.xacro"/>
+  <!-- Mesh/asset root (easy to swap if assets move) -->
+  <xacro:property name="asset_root" value="$(find 41068_ignition_bringup)/urdf_drone"/>
+  <!-- Camera placement helpers -->
   <xacro:property name="r200_cam_rgb_px" value="0.005"/>
   <xacro:property name="r200_cam_rgb_py" value="0.018"/>
@@ -24,5 +21,5 @@
         izz="3.328e-3"/>
     </inertial>
-    <!-- (Optional) simple collision box, keep commented unless you need it
+    <!-- (Optional) collision, leave commented unless you need it
     <collision name="collision">
       <origin xyz="-0.00424 0.00014 -0.00595" rpy="0 0 0"/>
@@ -120,4 +117,5 @@
   <link name="camera_depth_optical_frame"/>
   <!-- =============== Add Gazebo sensors + thermal cam =============== -->
+  <!-- You can pass visualize toggles here if you like -->
   <xacro:parrot_gz_extensions/>
 </robot>

Commit message: working 2

File: urdf_drone/parrot.urdf.xacro (robot description, xacro)
@@ -9,6 +9,6 @@
   <xacro:property name="r200_cam_rgb_pz" value="0.013"/>
   <xacro:property name="r200_cam_depth_offset" value="0.01"/>
-  <!-- Optional switch for thermal add-on (defaults ON) -->
-  <xacro:arg name="with_thermal" default="true"/>
+  <!-- Optional switch for thermal add-on (defaults ON)
+  <xacro:arg name="with_thermal" default="true"/> -->
   <!-- ================= Base geometry & frames (unchanged) ================= -->
   <link name="base_link">
@@ -118,7 +118,7 @@
   </joint>
   <link name="camera_depth_optical_frame"/>
-  <!-- ================= Thermal add-on (only addition) ================= -->
+  <!-- ================= Thermal add-on (only addition) =================
   <xacro:if value="$(arg with_thermal)">
-    <!-- Link + fixed joint off camera_link to follow the mast -->
+     Link + fixed joint off camera_link to follow the mast
     <link name="thermal_cam_link">
       <inertial>
@@ -136,9 +136,9 @@
       <child  link="thermal_cam_link"/>
       <origin xyz="0.06 0 0" rpy="0 0 0"/>
-      <!-- for nadir: rpy="0 -1.570796 0" -->
-    </joint>
-    <!-- Thermal sensors (topics match your detector/bridge) -->
+       for nadir: rpy="0 -1.570796 0"
+    </joint>-->
+    <!-- Thermal sensors (topics match your detector/bridge)
     <gazebo reference="thermal_cam_link">
-      <!-- 16-bit temperature image for processing -->
+       16-bit temperature image for processing
       <sensor name="parrot_thermal_l16" type="thermal">
         <always_on>1</always_on>
@@ -156,24 +156,5 @@
           <clip><near>0.05</near><far>100</far></clip>
         </camera>
-      </sensor>
-      <!-- 8-bit grayscale for easy viewing -->
-      <sensor name="parrot_thermal_l8" type="thermal">
-        <always_on>1</always_on>
-        <update_rate>15</update_rate>
-        <visualize>true</visualize>
-        <topic>/parrot/thermal/image_mono8</topic>
-        <gz_frame_id>thermal_cam_link</gz_frame_id>
-        <camera>
-          <horizontal_fov>1.047</horizontal_fov>
-          <image>
-            <width>320</width>
-            <height>240</height>
-            <format>L8</format>
-          </image>
-          <clip><near>0.05</near><far>100</far></clip>
-        </camera>
-      </sensor>
-    </gazebo>
-  </xacro:if>
+      </sensor> -->
   <!-- Note: All other sensors/plugins remain provided by parrot.gazebo.xacro include -->
 </robot>

Commit message: sorta working with thermal

File: urdf_drone/parrot.urdf.xacro (robot description, xacro)
@@ -1,15 +1,13 @@
-<?xml version="1.0" ?>
-<robot name="parrot" xmlns:xacro="http://ros.org/wiki/xacro">
-  <!-- Keep the original includes from the second package -->
+<?xml version="1.0"?>
+<robot name="parrot" xmlns:xacro="http://www.ros.org/wiki/xacro">
+  <!-- Includes (inside this package) -->
   <xacro:include filename="$(find 41068_ignition_bringup)/urdf_drone/common_properties.urdf.xacro"/>
   <xacro:include filename="$(find 41068_ignition_bringup)/urdf_drone/parrot.gazebo.xacro"/>
-  <!-- Properties (unchanged) -->
+  <!-- Camera placement helpers -->
   <xacro:property name="r200_cam_rgb_px" value="0.005"/>
   <xacro:property name="r200_cam_rgb_py" value="0.018"/>
   <xacro:property name="r200_cam_rgb_pz" value="0.013"/>
   <xacro:property name="r200_cam_depth_offset" value="0.01"/>
-  <!-- Optional switch for thermal add-on (defaults ON)
-  <xacro:arg name="with_thermal" default="true"/> -->
-  <!-- ================= Base geometry & frames (unchanged) ================= -->
+  <!-- ================= Base hull ================= -->
   <link name="base_link">
     <inertial>
@@ -49,5 +47,5 @@
     </visual>
   </link>
-  <!-- IMU frame -->
+  <!-- ================= IMU ================= -->
   <joint name="imu_joint" type="fixed">
     <parent link="base_link"/>
@@ -56,5 +54,5 @@
   </joint>
   <link name="imu_link"/>
-  <!-- Lidar frame -->
+  <!-- ================= Lidar puck (viz) ================= -->
   <joint name="scan_joint" type="fixed">
     <parent link="base_link"/>
@@ -74,9 +72,9 @@
     </inertial>
   </link>
-  <!-- Camera mast & frames -->
+  <!-- ================= Camera mast ================= -->
   <joint name="camera_joint" type="fixed">
-    <origin xyz="0.25 0.0 0.25" rpy="0 0.785398 0"/>
     <parent link="base_link"/>
     <child  link="camera_link"/>
+    <origin xyz="0.25 0.0 0.25" rpy="0 0.785398 0"/>
   </joint>
   <link name="camera_link">
@@ -92,69 +90,31 @@
     </visual>
   </link>
-  <!-- RGB frames -->
+  <!-- ================= RGB frames ================= -->
   <joint name="camera_rgb_joint" type="fixed">
-    <origin xyz="${r200_cam_rgb_px} ${r200_cam_rgb_py} ${r200_cam_rgb_pz}"/>
     <parent link="camera_link"/>
     <child  link="camera_rgb_frame"/>
+    <origin xyz="${r200_cam_rgb_px} ${r200_cam_rgb_py} ${r200_cam_rgb_pz}"/>
   </joint>
   <link name="camera_rgb_frame"/>
   <joint name="camera_rgb_optical_joint" type="fixed">
-    <origin xyz="0 0 0" rpy="-1.57 0 -1.57"/>
     <parent link="camera_rgb_frame"/>
     <child  link="camera_rgb_optical_frame"/>
+    <origin xyz="0 0 0" rpy="-1.57 0 -1.57"/>
   </joint>
   <link name="camera_rgb_optical_frame"/>
-  <!-- Depth frames -->
+  <!-- ================= Depth frames ================= -->
   <joint name="camera_depth_joint" type="fixed">
-    <origin xyz="${r200_cam_rgb_px} ${r200_cam_rgb_py + r200_cam_depth_offset} ${r200_cam_rgb_pz}"/>
     <parent link="camera_link"/>
     <child  link="camera_depth_frame"/>
+    <origin xyz="${r200_cam_rgb_px} ${r200_cam_rgb_py + r200_cam_depth_offset} ${r200_cam_rgb_pz}"/>
   </joint>
   <link name="camera_depth_frame"/>
   <joint name="camera_depth_optical_joint" type="fixed">
-    <origin xyz="0 0 0" rpy="-1.57 0 -1.57"/>
     <parent link="camera_depth_frame"/>
     <child  link="camera_depth_optical_frame"/>
+    <origin xyz="0 0 0" rpy="-1.57 0 -1.57"/>
   </joint>
   <link name="camera_depth_optical_frame"/>
-  <!-- ================= Thermal add-on (only addition) =================
-  <xacro:if value="$(arg with_thermal)">
-     Link + fixed joint off camera_link to follow the mast
-    <link name="thermal_cam_link">
-      <inertial>
-        <mass value="0.05"/>
-        <origin xyz="0 0 0"/>
-        <inertia ixx="1e-5" ixy="0" ixz="0" iyy="1e-5" iyz="0" izz="1e-5"/>
-      </inertial>
-      <visual name="thermal_cam_vis">
-        <origin xyz="0 0 0"/>
-        <geometry><box size="0.03 0.03 0.03"/></geometry>
-      </visual>
-    </link>
-    <joint name="thermal_cam_joint" type="fixed">
-      <parent link="camera_link"/>
-      <child  link="thermal_cam_link"/>
-      <origin xyz="0.06 0 0" rpy="0 0 0"/>
-       for nadir: rpy="0 -1.570796 0"
-    </joint>-->
-    <!-- Thermal sensors (topics match your detector/bridge)
-    <gazebo reference="thermal_cam_link">
-       16-bit temperature image for processing
-      <sensor name="parrot_thermal_l16" type="thermal">
-        <always_on>1</always_on>
-        <update_rate>15</update_rate>
-        <visualize>true</visualize>
-        <topic>/parrot/thermal/image_raw</topic>
-        <gz_frame_id>thermal_cam_link</gz_frame_id>
-        <camera>
-          <horizontal_fov>1.047</horizontal_fov>
-          <image>
-            <width>320</width>
-            <height>240</height>
-            <format>L16</format>
-          </image>
-          <clip><near>0.05</near><far>100</far></clip>
-        </camera>
-      </sensor> -->
-  <!-- Note: All other sensors/plugins remain provided by parrot.gazebo.xacro include -->
+  <!-- ================= Gazebo sensors + thermal camera ================= -->
+  <xacro:parrot_gz_extensions/>
 </robot>
