Commit message: Update parrot.gazebo.xacro - merged existing with thermal
Backup is in backup folder

File: urdf_drone/parrot.gazebo.xacro (robot description, xacro)
@@ -1,173 +1,149 @@
 <?xml version="1.0"?>
-<robot name="parrot" xmlns:xacro="http://ros.org/wiki/xacro">
-  <xacro:arg name="laser_visual"  default="false" />
-  <xacro:arg name="camera_visual" default="false"/>
-  <xacro:arg name="imu_visual"    default="false"/>
-  <!-- <xacro:include filename="$(find 41068_ignition_bringup)/urdf/wheel.urdf.xacro"/> -->
-  <gazebo reference="imu_link">
-    <sensor type="imu" name="imu">
-      <always_on>true</always_on>
-      <visualize>$(arg imu_visual)</visualize>
-      <update_rate>100</update_rate>
-      <topic>model/husky/imu</topic>
-      <gz_frame_id>imu_link</gz_frame_id>
-      <imu>
-        <angular_velocity>
-          <x>
-            <noise type="gaussian">
-              <mean>0.0</mean>
-              <stddev>2e-4</stddev>
-              <bias_mean>0.0000075</bias_mean>
-              <bias_stddev>0.0000008</bias_stddev>
-            </noise>
-          </x>
-          <y>
-            <noise type="gaussian">
-              <mean>0.0</mean>
-              <stddev>2e-4</stddev>
-              <bias_mean>0.0000075</bias_mean>
-              <bias_stddev>0.0000008</bias_stddev>
-            </noise>
-          </y>
-          <z>
-            <noise type="gaussian">
-              <mean>0.0</mean>
-              <stddev>2e-4</stddev>
-              <bias_mean>0.0000075</bias_mean>
-              <bias_stddev>0.0000008</bias_stddev>
-            </noise>
-          </z>
-        </angular_velocity>
-        <linear_acceleration>
-          <x>
-            <noise type="gaussian">
-              <mean>0.0</mean>
-              <stddev>1.7e-2</stddev>
-              <bias_mean>0.1</bias_mean>
-              <bias_stddev>0.001</bias_stddev>
-            </noise>
-          </x>
-          <y>
-            <noise type="gaussian">
-              <mean>0.0</mean>
-              <stddev>1.7e-2</stddev>
-              <bias_mean>0.1</bias_mean>
-              <bias_stddev>0.001</bias_stddev>
-            </noise>
-          </y>
-          <z>
-            <noise type="gaussian">
-              <mean>0.0</mean>
-              <stddev>1.7e-2</stddev>
-              <bias_mean>0.1</bias_mean>
-              <bias_stddev>0.001</bias_stddev>
-            </noise>
-          </z>
-        </linear_acceleration>
-      </imu>
-      <plugin
-        filename="ignition-gazebo-imu-system"
-        name="ignition::gazebo::systems::Imu">
-      </plugin>
-    </sensor>
-    <material>Gazebo/Grey</material>
-  </gazebo>
-  <!-- Move base directly without faffing around with diff drive controllers -->
-  <gazebo>
-    <plugin
-      filename="ignition-gazebo-velocity-control-system"
-      name="ignition::gazebo::systems::VelocityControl">
-      <topic>model/husky/cmd_vel</topic>
-    </plugin>
-  </gazebo>
-  <!-- Publish odometry separately -->
-  <gazebo>
-    <plugin
-      filename="ignition-gazebo-odometry-publisher-system"
-      name="ignition::gazebo::systems::OdometryPublisher">
-      <topic>model/husky/odometry</topic>
-      <odom_publish_frequency>20</odom_publish_frequency>
-      <odom_frame>odom</odom_frame>
-      <robot_base_frame>base_link</robot_base_frame>
-      <dimensions>3</dimensions>
-    </plugin>
-  </gazebo>
-  <gazebo>
-    <plugin
-      filename="ignition-gazebo-joint-state-publisher-system"
-      name="ignition::gazebo::systems::JointStatePublisher">
-      <topic>model/husky/joint_states</topic>
-    </plugin>
-  </gazebo>
-  <!-- Lidar and cameras use the general Sensors plugin -->
-  <gazebo>
-    <plugin
-        filename="libignition-gazebo-sensors-system.so"
-        name="ignition::gazebo::systems::Sensors">
-    </plugin>
-  </gazebo>
-  <gazebo reference="base_scan">
-    <material>Gazebo/FlatBlack</material>
-    <sensor type="gpu_lidar" name="lidar">
-      <pose relative_to='base_scan'>0 0 0 0 0 0</pose>
-      <visualize>$(arg laser_visual)</visualize>
-      <topic>model/husky/scan</topic>
-      <update_rate>3</update_rate>
-      <gz_frame_id>base_scan</gz_frame_id>
-      <ray>
-        <scan>
-          <horizontal>
-            <samples>360</samples>
-            <resolution>1</resolution>
-            <min_angle>0.0</min_angle>
-            <max_angle>6.28319</max_angle>
-          </horizontal>
-        </scan>
-        <range>
-          <min>0.2</min>
-          <max>40</max>
-          <resolution>0.015</resolution>
-        </range>
-        <noise>
-          <type>gaussian</type>
-          <mean>0.0</mean>
-          <stddev>0.01</stddev>
-        </noise>
-      </ray>
-      <always_on>true</always_on>
-    </sensor>
-  </gazebo>
-  <gazebo reference="camera_link">
-    <sensor name="rgbd_camera" type="rgbd_camera">
-      <camera>
-        <horizontal_fov>2.0944</horizontal_fov>
-        <image>
-          <width>720</width>
-          <height>480</height>
-        </image>
-        <clip>
-          <near>0.1</near>
-          <far>40</far>
-        </clip>
-        <!-- depth_camera near/far clip seems to be ignored for some reason -->
-        <!--    We're using Ignition Gazebo Fortress, which uses sdf format 1.9: http://sdformat.org/tutorials?tut=roadmap -->
-        <!--    This takes the depth_camera parameter with near / far clip http://sdformat.org/spec?ver=1.4&elem=sensor  -->
-        <!-- We also use ign sensors v6 ( run ls | grep libignition-sensors in /usr/lib/x86_64-linux-gnu)-->
-        <!-- Looking at the source code, the sdf sets HasDepthCamera() and corresponding HasDepthNearClip() & HasDepthFarClip() which are used in RgbdCameraSensor.cc, so this should work? -->
-        <!--    SDF description of Camera: https://github.com/gazebosim/sdformat/blob/sdf9/src/Camera.cc#L598-->
-        <!--    Camera sensor source code: https://github.com/gazebosim/gz-sensors/blob/ign-sensors6/src/RgbdCameraSensor.cc#L311  -->
-        <depth_camera>
+<robot xmlns:xacro="http://www.ros.org/wiki/xacro">
+  <!-- Optional toggles for sensor visuals in the GUI -->
+  <xacro:property name="show_imu_visual"    value="false"/>
+  <xacro:property name="show_lidar_visual"  value="false"/>
+  <xacro:property name="show_camera_visual" value="false"/>
+  <!-- Macro that adds mounted sensors (RGBD + Thermal) to the Parrot -->
+  <xacro:macro name="parrot_gz_extensions" params="">
+    <!-- ================= IMU on imu_link (adds noise + visualize toggle) ================= -->
+    <gazebo reference="imu_link">
+      <sensor type="imu" name="parrot_imu">
+        <always_on>true</always_on>
+        <visualize>${show_imu_visual}</visualize>
+        <update_rate>100</update_rate>
+        <topic>/parrot/imu</topic>
+        <gz_frame_id>imu_link</gz_frame_id>
+        <!-- Noise model merged from teammate's file -->
+        <imu>
+          <angular_velocity>
+            <x><noise type="gaussian"><mean>0.0</mean><stddev>2e-4</stddev><bias_mean>7.5e-6</bias_mean><bias_stddev>8e-7</bias_stddev></noise></x>
+            <y><noise type="gaussian"><mean>0.0</mean><stddev>2e-4</stddev><bias_mean>7.5e-6</bias_mean><bias_stddev>8e-7</bias_stddev></noise></y>
+            <z><noise type="gaussian"><mean>0.0</mean><stddev>2e-4</stddev><bias_mean>7.5e-6</bias_mean><bias_stddev>8e-7</bias_stddev></noise></z>
+          </angular_velocity>
+          <linear_acceleration>
+            <x><noise type="gaussian"><mean>0.0</mean><stddev>1.7e-2</stddev><bias_mean>0.1</bias_mean><bias_stddev>0.001</bias_stddev></noise></x>
+            <y><noise type="gaussian"><mean>0.0</mean><stddev>1.7e-2</stddev><bias_mean>0.1</bias_mean><bias_stddev>0.001</bias_stddev></noise></y>
+            <z><noise type="gaussian"><mean>0.0</mean><stddev>1.7e-2</stddev><bias_mean>0.1</bias_mean><bias_stddev>0.001</bias_stddev></noise></z>
+          </linear_acceleration>
+        </imu>
+      </sensor>
+    </gazebo>
+    <!-- ================ GPU lidar on base_scan (adds noise + visualize) ================ -->
+    <gazebo reference="base_scan">
+      <sensor type="gpu_lidar" name="parrot_lidar">
+        <always_on>true</always_on>
+        <visualize>${show_lidar_visual}</visualize>
+        <update_rate>10</update_rate>
+        <topic>/parrot/scan</topic>
+        <gz_frame_id>base_scan</gz_frame_id>
+        <ray>
+          <scan>
+            <horizontal>
+              <samples>360</samples>
+              <resolution>1</resolution>
+              <min_angle>0.0</min_angle>
+              <max_angle>6.28319</max_angle>
+            </horizontal>
+          </scan>
+          <range>
+            <min>0.2</min>
+            <max>40</max>
+            <resolution>0.015</resolution>
+          </range>
+          <noise>
+            <type>gaussian</type>
+            <mean>0.0</mean>
+            <stddev>0.01</stddev>
+          </noise>
+        </ray>
+      </sensor>
+    </gazebo>
+    <!-- ============ RGBD camera mounted on camera_link (keeps your config + visualize) ============ -->
+    <gazebo reference="camera_link">
+      <sensor name="parrot_rgbd" type="rgbd_camera">
+        <always_on>1</always_on>
+        <visualize>${show_camera_visual}</visualize>
+        <update_rate>10</update_rate>
+        <!-- Base topic; Gazebo publishes /image, /depth_image, /points, /camera_info -->
+        <topic>/parrot/camera</topic>
+        <gz_frame_id>camera_link</gz_frame_id>
+        <camera>
+          <horizontal_fov>2.0944</horizontal_fov>
+          <image>
+            <width>720</width>
+            <height>480</height>
+          </image>
           <clip>
-            <near>0.4</near>
-            <far>10</far>
+            <near>0.1</near>
+            <far>40</far>
           </clip>
-        </depth_camera>
-      </camera>
-      <always_on>1</always_on>
-      <update_rate>3</update_rate> <!--10-->
-      <visualize>$(arg camera_visual)</visualize>
-      <topic>/model/husky/camera</topic>
-      <gz_frame_id>camera_link</gz_frame_id>
-    </sensor>
-  </gazebo>
+          <depth_camera>
+            <clip>
+              <near>0.4</near>
+              <far>10</far>
+            </clip>
+          </depth_camera>
+        </camera>
+      </sensor>
+    </gazebo>
+    <!-- ===== Thermal camera: link + joint so it follows the drone (your original) ===== -->
+    <link name="thermal_cam_link">
+      <inertial>
+        <mass value="0.05"/>
+        <origin xyz="0 0 0"/>
+        <inertia ixx="1e-5" ixy="0" ixz="0" iyy="1e-5" iyz="0" izz="1e-5"/>
+      </inertial>
+      <visual name="thermal_cam_vis">
+        <origin xyz="0 0 0"/>
+        <geometry><box size="0.03 0.03 0.03"/></geometry>
+      </visual>
+    </link>
+    <joint name="thermal_cam_joint" type="fixed">
+      <parent link="camera_link"/>
+      <child  link="thermal_cam_link"/>
+      <!-- forward offset from the mast; same orientation as camera_link -->
+      <origin xyz="0.06 0 0" rpy="0 0 0"/>
+      <!-- for a nadir (down-looking) camera, use rpy="0 -1.570796 0" -->
+    </joint>
+    <!-- ============ Thermal sensors on thermal_cam_link (your L16 + L8 pair) ============ -->
+    <gazebo reference="thermal_cam_link">
+      <!-- 16-bit temperature image (good for processing) -->
+      <sensor name="parrot_thermal_l16" type="thermal">
+        <always_on>1</always_on>
+        <update_rate>15</update_rate>
+        <visualize>true</visualize>
+        <topic>/parrot/thermal/image_raw</topic>
+        <gz_frame_id>thermal_cam_link</gz_frame_id>
+        <camera>
+          <horizontal_fov>1.047</horizontal_fov>
+          <image>
+            <width>320</width>
+            <height>240</height>
+            <format>L16</format>
+          </image>
+          <clip><near>0.05</near><far>100</far></clip>
+        </camera>
+      </sensor>
+      <!-- 8-bit grayscale (easy to view in the GUI) -->
+      <sensor name="parrot_thermal_l8" type="thermal">
+        <always_on>1</always_on>
+        <update_rate>15</update_rate>
+        <visualize>true</visualize>
+        <topic>/parrot/thermal/image_mono8</topic>
+        <gz_frame_id>thermal_cam_link</gz_frame_id>
+        <camera>
+          <horizontal_fov>1.047</horizontal_fov>
+          <image>
+            <width>320</width>
+            <height>240</height>
+            <format>L8</format>
+          </image>
+          <clip><near>0.05</near><far>100</far></clip>
+        </camera>
+      </sensor>
+    </gazebo>
+    <!-- NOTE: No per-model Sensors/Velocity/Odom/JointState plugins here.
+         Sensors are driven by the world-level gz-sim-sensors-system you already load. -->
+  </xacro:macro>
 </robot>
