Commit message: Add files via upload
With thermal linkages

File: urdf_drone/parrot.gazebo.xacro (robot description, xacro)
@@ -1,173 +1,57 @@
-<?xml version="1.0"?>
-<robot name="parrot" xmlns:xacro="http://ros.org/wiki/xacro">
-  <xacro:arg name="laser_visual"  default="false" />
-  <xacro:arg name="camera_visual" default="false"/>
-  <xacro:arg name="imu_visual"    default="false"/>
-  <!-- <xacro:include filename="$(find 41068_ignition_bringup)/urdf/wheel.urdf.xacro"/> -->
-  <gazebo reference="imu_link">
-    <sensor type="imu" name="imu">
-      <always_on>true</always_on>
-      <visualize>$(arg imu_visual)</visualize>
-      <update_rate>100</update_rate>
-      <topic>model/husky/imu</topic>
-      <gz_frame_id>imu_link</gz_frame_id>
-      <imu>
-        <angular_velocity>
-          <x>
-            <noise type="gaussian">
-              <mean>0.0</mean>
-              <stddev>2e-4</stddev>
-              <bias_mean>0.0000075</bias_mean>
-              <bias_stddev>0.0000008</bias_stddev>
-            </noise>
-          </x>
-          <y>
-            <noise type="gaussian">
-              <mean>0.0</mean>
-              <stddev>2e-4</stddev>
-              <bias_mean>0.0000075</bias_mean>
-              <bias_stddev>0.0000008</bias_stddev>
-            </noise>
-          </y>
-          <z>
-            <noise type="gaussian">
-              <mean>0.0</mean>
-              <stddev>2e-4</stddev>
-              <bias_mean>0.0000075</bias_mean>
-              <bias_stddev>0.0000008</bias_stddev>
-            </noise>
-          </z>
-        </angular_velocity>
-        <linear_acceleration>
-          <x>
-            <noise type="gaussian">
-              <mean>0.0</mean>
-              <stddev>1.7e-2</stddev>
-              <bias_mean>0.1</bias_mean>
-              <bias_stddev>0.001</bias_stddev>
-            </noise>
-          </x>
-          <y>
-            <noise type="gaussian">
-              <mean>0.0</mean>
-              <stddev>1.7e-2</stddev>
-              <bias_mean>0.1</bias_mean>
-              <bias_stddev>0.001</bias_stddev>
-            </noise>
-          </y>
-          <z>
-            <noise type="gaussian">
-              <mean>0.0</mean>
-              <stddev>1.7e-2</stddev>
-              <bias_mean>0.1</bias_mean>
-              <bias_stddev>0.001</bias_stddev>
-            </noise>
-          </z>
-        </linear_acceleration>
-      </imu>
-      <plugin
-        filename="ignition-gazebo-imu-system"
-        name="ignition::gazebo::systems::Imu">
-      </plugin>
-    </sensor>
-    <material>Gazebo/Grey</material>
-  </gazebo>
-  <!-- Move base directly without faffing around with diff drive controllers -->
-  <gazebo>
-    <plugin
-      filename="ignition-gazebo-velocity-control-system"
-      name="ignition::gazebo::systems::VelocityControl">
-      <topic>model/husky/cmd_vel</topic>
-    </plugin>
-  </gazebo>
-  <!-- Publish odometry separately -->
-  <gazebo>
-    <plugin
-      filename="ignition-gazebo-odometry-publisher-system"
-      name="ignition::gazebo::systems::OdometryPublisher">
-      <topic>model/husky/odometry</topic>
-      <odom_publish_frequency>20</odom_publish_frequency>
-      <odom_frame>odom</odom_frame>
-      <robot_base_frame>base_link</robot_base_frame>
-      <dimensions>3</dimensions>
-    </plugin>
-  </gazebo>
-  <gazebo>
-    <plugin
-      filename="ignition-gazebo-joint-state-publisher-system"
-      name="ignition::gazebo::systems::JointStatePublisher">
-      <topic>model/husky/joint_states</topic>
-    </plugin>
-  </gazebo>
-  <!-- Lidar and cameras use the general Sensors plugin -->
-  <gazebo>
-    <plugin
-        filename="libignition-gazebo-sensors-system.so"
-        name="ignition::gazebo::systems::Sensors">
-    </plugin>
-  </gazebo>
-  <gazebo reference="base_scan">
-    <material>Gazebo/FlatBlack</material>
-    <sensor type="gpu_lidar" name="lidar">
-      <pose relative_to='base_scan'>0 0 0 0 0 0</pose>
-      <visualize>$(arg laser_visual)</visualize>
-      <topic>model/husky/scan</topic>
-      <update_rate>3</update_rate>
-      <gz_frame_id>base_scan</gz_frame_id>
-      <ray>
-        <scan>
-          <horizontal>
-            <samples>360</samples>
-            <resolution>1</resolution>
-            <min_angle>-1.17</min_angle>
-            <max_angle>1.17</max_angle>
-          </horizontal>
-        </scan>
-        <range>
-          <min>0.2</min>
-          <max>15</max>
-          <resolution>0.015</resolution>
-        </range>
-        <noise>
-          <type>gaussian</type>
-          <mean>0.0</mean>
-          <stddev>0.01</stddev>
-        </noise>
-      </ray>
-      <always_on>true</always_on>
-    </sensor>
-  </gazebo>
-  <gazebo reference="camera_link">
-    <sensor name="rgbd_camera" type="rgbd_camera">
-      <camera>
-        <horizontal_fov>2.0944</horizontal_fov>
-        <image>
-          <width>720</width>
-          <height>480</height>
-        </image>
-        <clip>
-          <near>0.1</near>
-          <far>40</far>
-        </clip>
-        <!-- depth_camera near/far clip seems to be ignored for some reason -->
-        <!--    We're using Ignition Gazebo Fortress, which uses sdf format 1.9: http://sdformat.org/tutorials?tut=roadmap -->
-        <!--    This takes the depth_camera parameter with near / far clip http://sdformat.org/spec?ver=1.4&elem=sensor  -->
-        <!-- We also use ign sensors v6 ( run ls | grep libignition-sensors in /usr/lib/x86_64-linux-gnu)-->
-        <!-- Looking at the source code, the sdf sets HasDepthCamera() and corresponding HasDepthNearClip() & HasDepthFarClip() which are used in RgbdCameraSensor.cc, so this should work? -->
-        <!--    SDF description of Camera: https://github.com/gazebosim/sdformat/blob/sdf9/src/Camera.cc#L598-->
-        <!--    Camera sensor source code: https://github.com/gazebosim/gz-sensors/blob/ign-sensors6/src/RgbdCameraSensor.cc#L311  -->
-        <depth_camera>
-          <clip>
-            <near>0.4</near>
-            <far>10</far>
-          </clip>
-        </depth_camera>
-      </camera>
-      <always_on>1</always_on>
-      <update_rate>3</update_rate> <!--10-->
-      <visualize>$(arg camera_visual)</visualize>
-      <topic>/model/husky/camera</topic>
-      <gz_frame_id>camera_link</gz_frame_id>
-    </sensor>
-  </gazebo>
-</robot>
+<!-- ==== Thermal camera: link + joint so it follows the drone (non-destructive add) ==== -->
+<link name="thermal_cam_link">
+  <inertial>
+    <mass value="0.05"/>
+    <origin xyz="0 0 0"/>
+    <inertia ixx="1e-5" ixy="0" ixz="0" iyy="1e-5" iyz="0" izz="1e-5"/>
+  </inertial>
+  <!-- tiny visual so you can see the sensor position -->
+  <visual name="thermal_cam_vis">
+    <origin xyz="0 0 0"/>
+    <geometry><box size="0.03 0.03 0.03"/></geometry>
+  </visual>
+</link>
+<joint name="thermal_cam_joint" type="fixed">
+  <parent link="camera_link"/>
+  <child  link="thermal_cam_link"/>
+  <!-- forward offset from the mast; same orientation as camera_link -->
+  <origin xyz="0.06 0 0" rpy="0 0 0"/>
+  <!-- for a nadir (down-looking) camera, use rpy="0 -1.570796 0" -->
+</joint>
+<!-- Two thermal sensors publishing L16 (for processing) and L8 (for viewing) -->
+<gazebo reference="thermal_cam_link">
+  <!-- 16-bit temperature image -->
+  <sensor name="parrot_thermal_l16" type="thermal">
+    <always_on>1</always_on>
+    <update_rate>15</update_rate>
+    <visualize>true</visualize>
+    <topic>/parrot/thermal/image_raw</topic>
+    <gz_frame_id>thermal_cam_link</gz_frame_id>
+    <camera>
+      <horizontal_fov>1.047</horizontal_fov>
+      <image>
+        <width>320</width>
+        <height>240</height>
+        <format>L16</format>
+      </image>
+      <clip><near>0.05</near><far>100</far></clip>
+    </camera>
+  </sensor>
+  <!-- 8-bit grayscale (easy to view in the GUI) -->
+  <sensor name="parrot_thermal_l8" type="thermal">
+    <always_on>1</always_on>
+    <update_rate>15</update_rate>
+    <visualize>true</visualize>
+    <topic>/parrot/thermal/image_mono8</topic>
+    <gz_frame_id>thermal_cam_link</gz_frame_id>
+    <camera>
+      <horizontal_fov>1.047</horizontal_fov>
+      <image>
+        <width>320</width>
+        <height>240</height>
+        <format>L8</format>
+      </image>
+      <clip><near>0.05</near><far>100</far></clip>
+    </camera>
+  </sensor>
+</gazebo>

File: urdf_drone/parrot.urdf.xacro (robot description, xacro)
@@ -1,25 +1,22 @@
 <?xml version="1.0" ?>
 <robot name="parrot" xmlns:xacro="http://ros.org/wiki/xacro">
+  <!-- Keep the original includes from the second package -->
   <xacro:include filename="$(find 41068_ignition_bringup)/urdf_drone/common_properties.urdf.xacro"/>
   <xacro:include filename="$(find 41068_ignition_bringup)/urdf_drone/parrot.gazebo.xacro"/>
+  <!-- Properties (unchanged) -->
   <xacro:property name="r200_cam_rgb_px" value="0.005"/>
   <xacro:property name="r200_cam_rgb_py" value="0.018"/>
   <xacro:property name="r200_cam_rgb_pz" value="0.013"/>
   <xacro:property name="r200_cam_depth_offset" value="0.01"/>
-  <!-- Main link -->
+  <!-- Optional switch for thermal add-on (defaults ON) -->
+  <xacro:arg name="with_thermal" default="true"/>
+  <!-- ================= Base geometry & frames (unchanged) ================= -->
   <link name="base_link">
     <inertial>
       <origin xyz="0 0 0" rpy="0 0 0"/>
-      <mass value="0.503"/> <!-- kg -->
+      <mass value="0.503"/>
       <inertia ixx="1.805e-3" ixy="-8.619e-7" ixz="1.555e-5"
-               iyy="1.764e-3" iyz="3.595e-7"
-               izz="3.328e-3" />
+               iyy="1.764e-3" iyz="3.595e-7" izz="3.328e-3"/>
     </inertial>
-<!--     <collision name="collision">
-      <origin xyz="-0.00424 0.00014 -0.00595" rpy="0 0 0"/>
-      <geometry>
-        <box size="0.5 0.5 0.2"/>
-      </geometry>
-    </collision> -->
     <visual name="hull">
       <geometry>
@@ -28,5 +25,5 @@
     </visual>
     <visual name="propeller_rr">
-      <origin xyz="-0.09035 -0.11423 -0.00501" rpy="0 0 0"/>
+      <origin xyz="-0.09035 -0.11423 -0.00501"/>
       <geometry>
         <mesh filename="file://$(find 41068_ignition_bringup)/urdf_drone/meshes/propeller_rr.dae"/>
@@ -34,5 +31,5 @@
     </visual>
     <visual name="propeller_rl">
-      <origin xyz="0.09035 0.11452 -0.00501" rpy="0 0 0"/>
+      <origin xyz="0.09035 0.11452 -0.00501"/>
       <geometry>
         <mesh filename="file://$(find 41068_ignition_bringup)/urdf_drone/meshes/propeller_rl.dae"/>
@@ -40,5 +37,5 @@
     </visual>
     <visual name="propeller_fr">
-      <origin xyz="0.08456 -0.11435 -0.00501" rpy="0 0 0"/>
+      <origin xyz="0.08456 -0.11435 -0.00501"/>
       <geometry>
         <mesh filename="file://$(find 41068_ignition_bringup)/urdf_drone/meshes/propeller_fr.dae"/>
@@ -46,5 +43,5 @@
     </visual>
     <visual name="propeller_fl">
-      <origin xyz="0.08456 0.11463 -0.00501" rpy="0 0 0"/>
+      <origin xyz="0.08456 0.11463 -0.00501"/>
       <geometry>
         <mesh filename="file://$(find 41068_ignition_bringup)/urdf_drone/meshes/propeller_fl.dae"/>
@@ -52,56 +49,52 @@
     </visual>
   </link>
+  <!-- IMU frame -->
   <joint name="imu_joint" type="fixed">
     <parent link="base_link"/>
-    <child link="imu_link"/>
-    <origin xyz="0.0 0 0.068" rpy="0 0 0"/>
+    <child  link="imu_link"/>
+    <origin xyz="0.0 0 0.068"/>
   </joint>
   <link name="imu_link"/>
+  <!-- Lidar frame -->
   <joint name="scan_joint" type="fixed">
     <parent link="base_link"/>
-    <child link="base_scan"/>
-    <origin xyz="0 0 0.2" rpy="0 0 0"/>
+    <child  link="base_scan"/>
+    <origin xyz="0 0 0.2"/>
   </joint>
   <link name="base_scan">
     <visual>
-      <origin xyz="0 0 0" rpy="0 0 0"/>
-      <geometry>
-        <cylinder length="0.04" radius="0.09"/>
-      </geometry>
+      <origin xyz="0 0 0"/>
+      <geometry><cylinder length="0.04" radius="0.09"/></geometry>
       <material name="dark"/>
     </visual>
     <inertial>
-      <mass value="0" />
-      <origin xyz="0 0 0" />
-      <inertia ixx="0.001" ixy="0.0" ixz="0.0"
-               iyy="0.001" iyz="0.0"
-               izz="0.001" />
+      <mass value="0"/>
+      <origin xyz="0 0 0"/>
+      <inertia ixx="0.001" ixy="0.0" ixz="0.0" iyy="0.001" iyz="0.0" izz="0.001"/>
     </inertial>
   </link>
+  <!-- Camera mast & frames -->
   <joint name="camera_joint" type="fixed">
-    <origin xyz="0.25 0.0 0.25" rpy="0 0.785398 0"/> <!-- 0.5 0.0 0.9 -->
+    <origin xyz="0.25 0.0 0.25" rpy="0 0.785398 0"/>
     <parent link="base_link"/>
-    <child link="camera_link"/>
+    <child  link="camera_link"/>
   </joint>
   <link name="camera_link">
     <visual>
-     <origin xyz="0 0 0" rpy="0 0 0"/>
-      <geometry>
-        <box size="0.02 0.08 0.05"/>
-      </geometry>
+      <origin xyz="0 0 0"/>
+      <geometry><box size="0.02 0.08 0.05"/></geometry>
       <material name="dark"/>
     </visual>
     <visual>
-     <origin xyz="0.015 0 0" rpy="0 1.57 0"/>
-      <geometry>
-        <cylinder length="0.03" radius="0.02"/>
-      </geometry>
+      <origin xyz="0.015 0 0" rpy="0 1.57 0"/>
+      <geometry><cylinder length="0.03" radius="0.02"/></geometry>
       <material name="dark"/>
     </visual>
   </link>
+  <!-- RGB frames -->
   <joint name="camera_rgb_joint" type="fixed">
-    <origin xyz="${r200_cam_rgb_px} ${r200_cam_rgb_py} ${r200_cam_rgb_pz}" rpy="0 0 0"/>
+    <origin xyz="${r200_cam_rgb_px} ${r200_cam_rgb_py} ${r200_cam_rgb_pz}"/>
     <parent link="camera_link"/>
-    <child link="camera_rgb_frame"/>
+    <child  link="camera_rgb_frame"/>
   </joint>
   <link name="camera_rgb_frame"/>
@@ -109,11 +102,12 @@
     <origin xyz="0 0 0" rpy="-1.57 0 -1.57"/>
     <parent link="camera_rgb_frame"/>
-    <child link="camera_rgb_optical_frame"/>
+    <child  link="camera_rgb_optical_frame"/>
   </joint>
   <link name="camera_rgb_optical_frame"/>
+  <!-- Depth frames -->
   <joint name="camera_depth_joint" type="fixed">
-    <origin xyz="${r200_cam_rgb_px} ${r200_cam_rgb_py + r200_cam_depth_offset} ${r200_cam_rgb_pz}" rpy="0 0 0"/>
+    <origin xyz="${r200_cam_rgb_px} ${r200_cam_rgb_py + r200_cam_depth_offset} ${r200_cam_rgb_pz}"/>
     <parent link="camera_link"/>
-    <child link="camera_depth_frame"/>
+    <child  link="camera_depth_frame"/>
   </joint>
   <link name="camera_depth_frame"/>
@@ -121,6 +115,65 @@
     <origin xyz="0 0 0" rpy="-1.57 0 -1.57"/>
     <parent link="camera_depth_frame"/>
-    <child link="camera_depth_optical_frame"/>
+    <child  link="camera_depth_optical_frame"/>
   </joint>
   <link name="camera_depth_optical_frame"/>
+  <!-- ================= Thermal add-on (only addition) ================= -->
+  <xacro:if value="$(arg with_thermal)">
+    <!-- Link + fixed joint off camera_link to follow the mast -->
+    <link name="thermal_cam_link">
+      <inertial>
+        <mass value="0.05"/>
+        <origin xyz="0 0 0"/>
+        <inertia ixx="1e-5" ixy="0" ixz="0" iyy="1e-5" iyz="0" izz="1e-5"/>
+      </inertial>
+      <visual name="thermal_cam_vis">
+        <origin xyz="0 0 0"/>
+        <geometry><box size="0.03 0.03 0.03"/></geometry>
+      </visual>
+    </link>
+    <joint name="thermal_cam_joint" type="fixed">
+      <parent link="camera_link"/>
+      <child  link="thermal_cam_link"/>
+      <origin xyz="0.06 0 0" rpy="0 0 0"/>
+      <!-- for nadir: rpy="0 -1.570796 0" -->
+    </joint>
+    <!-- Thermal sensors (topics match your detector/bridge) -->
+    <gazebo reference="thermal_cam_link">
+      <!-- 16-bit temperature image for processing -->
+      <sensor name="parrot_thermal_l16" type="thermal">
+        <always_on>1</always_on>
+        <update_rate>15</update_rate>
+        <visualize>true</visualize>
+        <topic>/parrot/thermal/image_raw</topic>
+        <gz_frame_id>thermal_cam_link</gz_frame_id>
+        <camera>
+          <horizontal_fov>1.047</horizontal_fov>
+          <image>
+            <width>320</width>
+            <height>240</height>
+            <format>L16</format>
+          </image>
+          <clip><near>0.05</near><far>100</far></clip>
+        </camera>
+      </sensor>
+      <!-- 8-bit grayscale for easy viewing -->
+      <sensor name="parrot_thermal_l8" type="thermal">
+        <always_on>1</always_on>
+        <update_rate>15</update_rate>
+        <visualize>true</visualize>
+        <topic>/parrot/thermal/image_mono8</topic>
+        <gz_frame_id>thermal_cam_link</gz_frame_id>
+        <camera>
+          <horizontal_fov>1.047</horizontal_fov>
+          <image>
+            <width>320</width>
+            <height>240</height>
+            <format>L8</format>
+          </image>
+          <clip><near>0.05</near><far>100</far></clip>
+        </camera>
+      </sensor>
+    </gazebo>
+  </xacro:if>
+  <!-- Note: All other sensors/plugins remain provided by parrot.gazebo.xacro include -->
 </robot>
